Commit message: Added gripper tool frame to have a proper tip frame

File: jaco_description/robots/standalone_arm.urdf.xacro (robot description, xacro)
@@ -14,4 +14,5 @@
 	xmlns:xacro="http://ros.org/wiki/xacro" name="jaco">
 	<xacro:include filename="$(find jaco_description)/urdf/jaco_arm.urdf.xacro" />
+	<xacro:property name="M_PI" value="3.1415926535897931" />
 	<link name="root">
 		<visual>
@@ -28,4 +29,29 @@
 		</collision>
 	</link>
+	 <joint name="jaco_gripper_tool_frame_joint" type="fixed">
+        <parent link="jaco_link_hand"/>
+        <child link="jaco_gripper_tool_frame"/>
+        <origin rpy="${-M_PI/2} ${M_PI/2} 0" xyz="0 0 -0.1"/>
+    </joint>
+    <link name="jaco_gripper_tool_frame">
+        <!-- This is the coordinate system of the tool (this is the position
+         used in IK etc., relative to the base frame); there is no actual
+         arm part attached to this link -->
+        <!-- The visual and collision are a workaround for a bug when a object is
+     attached to a link without collision geometry the object's collisions are ignored-->
+        <!--<visual>
+            <origin rpy="0 0 0" xyz="0 0 0"/>
+            <geometry>
+                <box size="0.001 0.001 0.001"/>
+            </geometry>
+            <material name="black"/>
+        </visual>
+        <collision>
+            <origin rpy="0 0 0" xyz="0 0 0"/>
+            <geometry>
+                <box size="0.001 0.001 0.001"/>
+            </geometry>
+        </collision>-->
+    </link>
 	<xacro:jaco_arm parent="root" xyz="0 0 0" rpy="0 0 0" />
 </robot>

Commit message: renamed root to jaco_base_link

File: jaco_description/robots/standalone_arm.urdf.xacro (robot description, xacro)
@@ -15,5 +15,5 @@
 	<xacro:include filename="$(find jaco_description)/urdf/jaco_arm.urdf.xacro" />
 	<xacro:property name="M_PI" value="3.1415926535897931" />
-	<link name="root">
+	<link name="jaco_base_link">
 		<visual>
 			<origin xyz="0 0 0" rpy="0 0 0" />
@@ -54,4 +54,4 @@
         </collision>-->
     </link>
-	<xacro:jaco_arm parent="root" xyz="0 0 0" rpy="0 0 0" />
+	<xacro:jaco_arm parent="jaco_base_link" xyz="0 0 0" rpy="0 0 0" />
 </robot>
